File: hardware/nfc_sense.kicad_pcb (KiCad board)
At the start: 2 copper layers, 18.6 x 43.1 mm, 23 parts, among them U1 TMP117AIYBGR, U2 RF430CL330HIRGTR‎, U3 ATtiny1626-MFR

Commit message: init own repo
Parts:
- removed QR_ref1: TestPoint, unsurv_offline_pcb_footprints:QR_shop
- removed U1: TMP117AIYBGR, unsurv_offline_pcb_footprints:TMP117
- removed VCC1: TestPoint, TestPoint:TestPoint_Pad_D1.0mm
- added TP5: TestPoint, TestPoint:TestPoint_Pad_D1.0mm, B.Cu at (125.1, 47.6)
- added U4: TMP117AIYBGR, easyeda2kicad:DSBGA-6_L1.5-W1.0-R3-C2-P0.40-TL, F.Cu at (129.5, 38.7)
- U2: footprint unsurv_offline_pcb_footprints:RF430_3x3mm_noBCu -> easyeda2kicad:VQFN-16_L3.0-W3.0-P0.50-BL-EP1.7
- U3: footprint Package_DFN_QFN:VQFN-20-1EP_3x3mm_P0.4mm_EP1.7x1.7mm -> easyeda2kicad:QFN-20_L3.0-W3.0-P0.40-BL-EP1.7
- turned U2 to 0 degrees
- turned U3 to -90 degrees
- renumbered GND1 to TP6, UPDI1 to TP7
Other:
- board text added: "Patrick Lermer v0.8 unsurv/NFC_temp 03/24"
- board text removed: "v 0.8 pre-production 03/24"
