File: hardware/nfc_sense.kicad_sch (KiCad schematic)
At the start: 23 parts, among them U1 TMP117AIYBGR, U2 RF430CL330HIRGTR‎, U3 ATtiny1626-MFR

Commit message: init own repo
Parts:
- removed QR_ref1: TestPoint, unsurv_offline_pcb_footprints:QR_shop, symbol Connector:TestPoint
- removed U1: TMP117AIYBGR, unsurv_offline_pcb_footprints:TMP117, symbol dk_Temperature-Sensors-Analog-and-Digital-Output:TMP112AIDRLT
- removed VCC1: TestPoint, TestPoint:TestPoint_Pad_D1.0mm, symbol Connector:TestPoint
- added TP5: TestPoint, TestPoint:TestPoint_Pad_D1.0mm, symbol Connector:TestPoint
- added U4: TMP117AIYBGR, easyeda2kicad:DSBGA-6_L1.5-W1.0-R3-C2-P0.40-TL, symbol easyeda2kicad:TMP117AIYBGR
- U2: footprint unsurv_offline_pcb_footprints:RF430_3x3mm_noBCu -> easyeda2kicad:VQFN-16_L3.0-W3.0-P0.50-BL-EP1.7
- U3: footprint Package_DFN_QFN:VQFN-20-1EP_3x3mm_P0.4mm_EP1.7x1.7mm -> easyeda2kicad:QFN-20_L3.0-W3.0-P0.40-BL-EP1.7
- renumbered GND1 to TP6, UPDI1 to TP7
Connections:
- net GND: now also U4.B2 (GND), U4.C1 (ADD0)
- net SCL: now also U4.A2 (SCL)
- net SDA: now also U4.A1 (SDA)
- net VCC: now also TP5.1, U4.B1 (V+)
- no-connect marks 0 -> 11
Other:
- moved on the sheet: C7, TP2, U3
